File: mgr_board.kicad_sch (KiCad schematic)
At the start: 24 parts, among them IC1 MCP48CVB08-20E_ST, J1 DC_DC_Buck_converter_module, J2 Screw_Terminal_2_P5.00mm, J3 SD Card SPI Module

Commit message: small changes
Parts:
- C9: footprint Capacitor_SMD:C_1206_3216Metric_Pad1.33x1.80mm_HandSolder -> Capacitor_THT:C_Disc_D3.0mm_W2.0mm_P2.50mm
Other:
- moved on the sheet: C10, C12, C13, J1, J2, J3
