File: mgr_board.kicad_sch (KiCad schematic)
At the start: 2 parts

Commit message: draft
Parts:
- added ADC0: ADS1148QPWRQ1, ADC:SOP65P640X120-28N, symbol ADS1148QPWRQ1:ADS1148QPWRQ1
- added C1, C2, C3, C4: ?, Capacitor_THT:C_Disc_D3.0mm_W2.0mm_P2.50mm, symbol PCM_SL_Devices:Capacitor_NP
- added D1: ?, 4ms_Diode:D_SMA, symbol PCM_4ms_Diode:B140-E3
- added IC1: MCP48CVB08-20E_ST, DAC:SOP65P640X120-20N, symbol MCP48CVB08-20E_ST:MCP48CVB08-20E_ST
- added IC2: A6214KLKTR-T, LED_Driver:SOP100P600X165-11N, symbol A6214KLKTR-T:A6214KLKTR-T
- added L1: L, symbol Device:L
- added LED0: JR5050CWT-E-B50EB0000-N0000001, JR5050CWTEB50EB0000N0000001, symbol JR5050CWT-E-B50EB0000-N0000001:JR5050CWT-E-B50EB0000-N0000001
- added R1, R2, R3: ?, Resistor_THT:R_Axial_DIN0207_L6.3mm_D2.5mm_P10.16mm_Horizontal, symbol PCM_SL_Resistors:Resistor
- TH1: value Thermistor_NTC -> NTC
Connections:
- net +3V3: now also R1.2; no longer A1.31 (ADC0/GP26), TH1.1
- net GND: now also ADC0.2 (DGND), ADC0.21 (AVSS), C1.1, C2.1, C4.1, D1.2 (A), IC2.11 (GND_2), IC2.6 (GND_1), LED0.1 (K), LED0.3 (EP)
- net MISO: now reaches A1.1 (GP0)
- net MISO: now also ADC0.26 (DOUT/~{DRDY}), IC1.17 (SDO)
- net ADC0_CS: now reaches A1.2 (GP1)
- net ADC0_CS: now also ADC0.24 (~{CS})
- net PWM_0: now reaches A1.34 (ADC2/GP28)
- net PWM_0: now also IC2.3 (EN/PWM)
- net SCL: now reaches A1.4 (GP2)
- net SCL: now also ADC0.28 (SCLK), IC1.18 (SCK)
- net MOSI: now reaches A1.5 (GP3)
- net MOSI: now also ADC0.27 (DIN), IC1.19 (SDI)
- new net: C4.2, IC2.4 (ADIM), IC2.5 (VCC)
- new net: C3.2, D1.1 (K), IC2.10 (SW), L1.1
- new net: IC2.2 (TON), R2.1
- new net: C3.1, IC2.9 (BOOT)
- new net +12V: C1.2, C2.2, IC2.1 (VIN), R2.2
- new net +5V: ADC0.1 (DVDD), ADC0.22 (AVDD)
- new net ADC_NTC: A1.31 (ADC0/GP26), R1.1, TH1.1
- new net DAC_CS: IC1.3 (~{CS})
- new net I_LED_0: ADC0.12 (AIN1/IEXC), IC2.8 (CSH), L1.2, R3.2
- new net LED_0: ADC0.11 (AIN0/IEXC), IC2.7 (CSL), LED0.2 (A), R3.1
Other:
- moved on the sheet: A1, TH1

Commit message: First board schematic version
Parts:
- removed C1, C2, C3, C4: ?, Capacitor_THT:C_Disc_D3.0mm_W2.0mm_P2.50mm, symbol PCM_SL_Devices:Capacitor_NP
- removed D1: ?, 4ms_Diode:D_SMA, symbol PCM_4ms_Diode:B140-E3
- removed IC2: A6214KLKTR-T, LED_Driver:SOP100P600X165-11N, symbol A6214KLKTR-T:A6214KLKTR-T
- removed L1: L, symbol Device:L
- removed LED0: JR5050CWT-E-B50EB0000-N0000001, JR5050CWTEB50EB0000N0000001, symbol JR5050CWT-E-B50EB0000-N0000001:JR5050CWT-E-B50EB0000-N0000001
- removed R2, R3: ?, Resistor_THT:R_Axial_DIN0207_L6.3mm_D2.5mm_P10.16mm_Horizontal, symbol PCM_SL_Resistors:Resistor
- added ADC1, ADC2: ADS1148QPWRQ1, ADC:SOP65P640X120-28N, symbol ADS1148QPWRQ1:ADS1148QPWRQ1
- added C10, C11, C9: 1 uF, Capacitor_SMD:C_1206_3216Metric_Pad1.33x1.80mm_HandSolder, symbol PCM_SL_Devices:Capacitor_NP
- added J1: DC_DC_Buck_converter_module, Connector_PinHeader_2.54mm:PinHeader_1x03_P2.54mm_Vertical, symbol PCM_SL_Pin_Headers:PINHD_1x3_Male
- added J2: Screw_Terminal_2_P5.00mm, Connector_Samtec_HPM_THT:Samtec_HPM-02-01-x-S_Straight_1x02_Pitch5.08mm, symbol PCM_SL_Screw_Terminal:Screw_Terminal_2_P5.00mm
- added J3: SD Card SPI Module, Connector_PinHeader_2.54mm:PinHeader_1x06_P2.54mm_Vertical, symbol PCM_4ms_Connector:Conn_01x06
- added R10, R8, R9: 10k, Resistor_SMD:R_1206_3216Metric_Pad1.30x1.75mm_HandSolder, symbol PCM_SL_Resistors:Resistor
- R1: value ? -> 1k; footprint Resistor_THT:R_Axial_DIN0207_L6.3mm_D2.5mm_P10.16mm_Horizontal -> Resistor_SMD:R_1206_3216Metric_Pad1.30x1.75mm_HandSolder
- TH1: value NTC -> NTC 2.2k; footprint (none) -> Resistor_SMD:R_0805_2012Metric_Pad1.20x1.40mm_HandSolder
Connections:
- net +12V: now also J1.1, J2.2
- net +3V3: now also ADC0.1 (DVDD), ADC0.22 (AVDD), ADC0.23 (START), IC1.2 (VDD), TH1.1, ADC1.1 (DVDD), ADC1.22 (AVDD), ADC1.23 (START), ADC2.1 (DVDD), ADC2.22 (AVDD), ADC2.23 (START), J3.2 (Pin_2), R10.2, R8.2, R9.2; no longer R1.2
- net +5V: now also A1.39 (VSYS), J1.3; no longer ADC0.1 (DVDD), ADC0.22 (AVDD)
- net ADC_NTC: now also R1.2, TH1.2; no longer R1.1, TH1.1
- net DAC_CS: now also A1.7 (GP5)
- net GND: now also ADC0.10 (VREFCOM), ADC0.3 (CLK), IC1.9 (VSS), R1.1, ADC1.10 (VREFCOM), ADC1.2 (DGND), ADC1.21 (AVSS), ADC1.3 (CLK), ADC2.10 (VREFCOM), ADC2.2 (DGND), ADC2.21 (AVSS), ADC2.3 (CLK), C10.2, C11.2, C9.2, J1.2, J2.1, J3.1 (Pin_1); no longer TH1.2
- net ADC1_DRDY: now reaches A1.10 (GP7)
- net ADC1_DRDY: now also ADC1.25 (~{DRDY})
- net ADC2_DRDY: now reaches A1.11 (GP8)
- net ADC2_DRDY: now also ADC2.25 (~{DRDY})
- net ADC1_CS: now reaches A1.12 (GP9)
- net ADC1_CS: now also ADC1.24 (~{CS})
- net SPI1_SCL: now reaches A1.14 (GP10)
- net SPI1_SCL: now also ADC1.28 (SCLK), ADC2.28 (SCLK)
- net SPI1_MOSI: now reaches A1.15 (GP11)
- net SPI1_MOSI: now also ADC1.27 (DIN), ADC2.27 (DIN)
- net SPI1_MISO: now reaches A1.16 (GP12)
- net SPI1_MISO: now also ADC1.26 (DOUT/~{DRDY}), ADC2.26 (DOUT/~{DRDY})
- net ADC2_CS: now reaches A1.17 (GP13)
- net ADC2_CS: now also ADC2.24 (~{CS})
- net SD_CS: now reaches A1.22 (GP17)
- net SD_CS: now also J3.6 (Pin_6)
- net PWM_5: now reaches A1.25 (GP19)
- net PWM_4: now reaches A1.26 (GP20)
- net PWM_3: now reaches A1.27 (GP21)
- net PWM_2: now reaches A1.29 (GP22)
- net PWM_1: now reaches A1.32 (ADC1/GP27)
- net ADC0_DRDY: now reaches A1.9 (GP6)
- net ADC0_DRDY: now also ADC0.25 (~{DRDY})
- net V_LED_2: now reaches ADC0.13 (AIN4/IEXC/GPIO4)
- net I_LED_2: now reaches ADC0.14 (AIN5/IEXC/GPIO5)
- net V_LED_3: now reaches ADC0.15 (AIN6/IEXC/GPIO6)
- net I_LED_3: now reaches ADC0.16 (AIN7/IEXC/GPIO7)
- net V_LED_1: now reaches ADC0.17 (AIN2/IEXC/GPIO2)
- net I_LED_1: now reaches ADC0.18 (AIN3/IEXC/GPIO3)
- net at ADC0.4 (~{RESET}): now also R8.1
- net at ADC0.9 (VREFOUT): now also C9.1
- net ADIM_7: now reaches IC1.12 (VOUT7)
- net ADIM_5: now reaches IC1.13 (VOUT5)
- net ADIM_3: now reaches IC1.14 (VOUT3)
- net ADIM_1: now reaches IC1.15 (VOUT1)
- net ADIM_0: now reaches IC1.5 (VOUT0)
- net ADIM_2: now reaches IC1.6 (VOUT2)
- net ADIM_4: now reaches IC1.7 (VOUT4)
- net ADIM_6: now reaches IC1.8 (VOUT6)
- net LED_0 renamed V_LED_0
- net MISO renamed SPI0_MISO
- net SPI0_MISO: now also J3.3 (Pin_3)
- net MOSI renamed SPI0_MOSI
- net SPI0_MOSI: now also J3.4 (Pin_4)
- net SCL renamed SPI0_SCL
- net SPI0_SCL: now also J3.5 (Pin_5)
- new net: ADC2.4 (~{RESET}), R10.1
- new net: ADC2.9 (VREFOUT), C11.1
- new net: ADC1.4 (~{RESET}), R9.1
- new net: ADC1.9 (VREFOUT), C10.1
- new net I_LED_10: ADC2.14 (AIN5/IEXC/GPIO5)
- new net I_LED_11: ADC2.16 (AIN7/IEXC/GPIO7)
- new net I_LED_4: ADC1.12 (AIN1/IEXC)
- new net I_LED_5: ADC1.18 (AIN3/IEXC/GPIO3)
- new net I_LED_6: ADC1.14 (AIN5/IEXC/GPIO5)
- new net I_LED_7: ADC1.16 (AIN7/IEXC/GPIO7)
- new net I_LED_8: ADC2.12 (AIN1/IEXC)
- new net I_LED_9: ADC2.18 (AIN3/IEXC/GPIO3)
- new net V_LED_10: ADC2.13 (AIN4/IEXC/GPIO4)
- new net V_LED_11: ADC2.15 (AIN6/IEXC/GPIO6)
- new net V_LED_4: ADC1.11 (AIN0/IEXC)
- new net V_LED_5: ADC1.17 (AIN2/IEXC/GPIO2)
- new net V_LED_6: ADC1.13 (AIN4/IEXC/GPIO4)
- new net V_LED_7: ADC1.15 (AIN6/IEXC/GPIO6)
- new net V_LED_8: ADC2.11 (AIN0/IEXC)
- new net V_LED_9: ADC2.17 (AIN2/IEXC/GPIO2)
- no-connect marks 0 -> 32
Other:
- added sheet LED_Power_Section_1 (LED_Power_Section_1.kicad_sch)
- added sheet LED_Section (LED_Section.kicad_sch)
- added sheet Led_Power_Section_2 (Led_Power_Section_2.kicad_sch)
- moved on the sheet: A1, ADC0, IC1

Commit message: reviewed
Parts:
- added C12: 100nF, symbol Device:C_Small
- added C13: 4,7uF, symbol Device:C_Small
Connections:
- net +3V3: no longer IC1.2 (VDD)
- net GND: now also C12.2, C13.2
- net V_LED_0 renamed LED_0
- new net: C12.1, C13.1, IC1.2 (VDD)
Other:
- sheet LED_Power_Section_1 ports: added I_LED_0, LED_0, PWM_0; removed none
- sheet LED_Section ports: added LED_0, LED_1, LED_10, LED_11, LED_2, LED_3, LED_4, LED_5, LED_6, LED_7, LED_8, LED_9; removed none
- note added: "1.ADC na jednego SPI, a reszte na drugiego 2.Popatrz jakie napięcie bedziesz mierzył i jakie max napiecie moze mierzyc ADC 3. Capy decoupling"
- note added: "WHERE IS BUCK CONVERTER"
- note added: "tu tez capy"
- moved on the sheet: IC1, J1, J2, J3

Commit message: fixing review suggestions
Parts:
- added C14, C15, C16, C17, C18, C19: 100nF, Capacitor_SMD:C_1206_3216Metric_Pad1.33x1.80mm_HandSolder, symbol Device:C_Small
- C12, C13: footprint (none) -> Capacitor_SMD:C_1206_3216Metric_Pad1.33x1.80mm_HandSolder
Connections:
- net +3V3: now also C12.1, C13.1, IC1.2 (VDD), C15.1, C16.1, C17.1; no longer ADC0.22 (AVDD), ADC0.23 (START), ADC1.22 (AVDD), ADC1.23 (START), ADC2.22 (AVDD), ADC2.23 (START)
- net +5V: now also ADC0.22 (AVDD), ADC0.23 (START), ADC0.5 (REFP0/GPIO0), ADC1.22 (AVDD), ADC1.23 (START), ADC1.5 (REFP0/GPIO0), ADC2.22 (AVDD), ADC2.23 (START), ADC2.5 (REFP0/GPIO0), C14.2, C18.2, C19.2
- net ADC1_CS: now also A1.7 (GP5); no longer A1.12 (GP9)
- net ADC2_CS: now also A1.22 (GP17); no longer A1.17 (GP13)
- net ADIM_0: now also IC1.8 (VOUT6); no longer IC1.5 (VOUT0)
- net ADIM_1: now also IC1.12 (VOUT7); no longer IC1.15 (VOUT1)
- net ADIM_2: now also IC1.7 (VOUT4); no longer IC1.6 (VOUT2)
- net ADIM_3: now also IC1.13 (VOUT5); no longer IC1.14 (VOUT3)
- net ADIM_4: now also IC1.6 (VOUT2); no longer IC1.7 (VOUT4)
- net ADIM_5: now also IC1.14 (VOUT3); no longer IC1.13 (VOUT5)
- net ADIM_6: now also IC1.5 (VOUT0); no longer IC1.8 (VOUT6)
- net ADIM_7: now also IC1.15 (VOUT1); no longer IC1.12 (VOUT7)
- net DAC_CS: now also A1.12 (GP9); no longer A1.7 (GP5)
- net GND: now also ADC0.6 (REFN0/GPIO1), ADC1.6 (REFN0/GPIO1), ADC2.6 (REFN0/GPIO1), C14.1, C15.2, C16.2, C17.2, C18.1, C19.1
- net SD_CS: now also A1.17 (GP13), J3.3 (Pin_3); no longer A1.22 (GP17), J3.6 (Pin_6)
- net SPI0_MISO: now also ADC1.26 (DOUT/~{DRDY}), ADC2.26 (DOUT/~{DRDY}); no longer ADC0.26 (DOUT/~{DRDY}), IC1.17 (SDO), J3.3 (Pin_3)
- net SPI0_MOSI: now also ADC1.27 (DIN), ADC2.27 (DIN); no longer ADC0.27 (DIN), IC1.19 (SDI), J3.4 (Pin_4)
- net SPI0_SCL: now also ADC1.28 (SCLK), ADC2.28 (SCLK); no longer ADC0.28 (SCLK), IC1.18 (SCK), J3.5 (Pin_5)
- net SPI1_MISO: now also IC1.19 (SDI), J3.6 (Pin_6); no longer ADC1.26 (DOUT/~{DRDY}), ADC2.26 (DOUT/~{DRDY})
- net SPI1_MOSI: now also IC1.17 (SDO), J3.5 (Pin_5); no longer ADC1.27 (DIN), ADC2.27 (DIN)
- net SPI1_SCL: now also IC1.18 (SCK), J3.4 (Pin_4); no longer ADC1.28 (SCLK), ADC2.28 (SCLK)
- net V_LED_1 renamed LED_1
- net V_LED_10 renamed LED_10
- net V_LED_11 renamed LED_11
- net V_LED_2 renamed LED_2
- net V_LED_3 renamed LED_3
- net V_LED_4 renamed LED_4
- net V_LED_5 renamed LED_5
- net V_LED_6 renamed LED_6
- net V_LED_7 renamed LED_7
- net V_LED_8 renamed LED_8
- net V_LED_9 renamed LED_9
- no-connect marks 32 -> 26
Other:
- sheet Led_Power_Section_2 ports: added ADIM_0, I_LED_6, LED_6; removed none
- note removed: "WHERE IS BUCK CONVERTER"
- moved on the sheet: ADC0, ADC1, ADC2, C10, C11, C12, C13, C9, IC1, R1, R10, R8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

Commit message: small changes
Parts:
- removed C10, C11, C9: 1 uF, Capacitor_SMD:C_1206_3216Metric_Pad1.33x1.80mm_HandSolder, symbol PCM_SL_Devices:Capacitor_NP
- added C10, C20, C9: 1 uF, Capacitor_SMD:C_1206_3216Metric_Pad1.33x1.80mm_HandSolder, symbol Device:C_Small
Connections:
- net GND: now also C10.2, C20.2, C9.2
- net at ADC2.9 (VREFOUT): now also C10.1
- net at ADC1.9 (VREFOUT): now also C9.1
- net at ADC0.9 (VREFOUT): now also C20.1
Other:
- moved on the sheet: C12, C13, J1, J2, J3

Commit message: first complete version schematics
Connections:
- net SPI0_MISO: now also ADC0.26 (DOUT/~{DRDY})
- net SPI0_MOSI: now also ADC0.27 (DIN)
- net SPI0_SCL: now also ADC0.28 (SCLK)
- net SPI1_MISO: now also IC1.17 (SDO); no longer IC1.19 (SDI)
- net SPI1_MOSI: now also IC1.19 (SDI); no longer IC1.17 (SDO)
Other:
- sheet LED_Power_Section_1 ports: added I_LED_1, I_LED_2, I_LED_3, I_LED_4, I_LED_5, LED_1, LED_2, LED_3, LED_4, LED_5, PWM_1, PWM_2, PWM_3, PWM_4, PWM_5; removed none
- sheet Led_Power_Section_2 ports: added ADIM_1, ADIM_2, ADIM_3, ADIM_4, ADIM_5, I_LED_10, I_LED_11, I_LED_7, I_LED_8, I_LED_9, LED_10, LED_11, LED_7, LED_8, LED_9; removed none
- note removed: "1.ADC na jednego SPI, a reszte na drugiego 2.Popatrz jakie napięcie bedziesz mierzył i jakie max napiecie moze mierzyc ADC 3. Capy decoupling"
- moved on the sheet: R1, TH1

Commit message: Changed footprints of passive elements, reviewed
Parts:
- removed C10, C20, C9: 1 uF, Capacitor_SMD:C_1206_3216Metric_Pad1.33x1.80mm_HandSolder, symbol Device:C_Small
- removed J1: DC_DC_Buck_converter_module, Connector_PinHeader_2.54mm:PinHeader_1x03_P2.54mm_Vertical, symbol PCM_SL_Pin_Headers:PINHD_1x3_Male
- removed J3: SD Card SPI Module, Connector_PinHeader_2.54mm:PinHeader_1x06_P2.54mm_Vertical, symbol PCM_4ms_Connector:Conn_01x06
- added C1: 4,7uF, Capacitor_SMD:C_0603_1608Metric_Pad1.08x0.95mm_HandSolder, symbol Device:C_Small
- added C2: 100nF, Capacitor_SMD:C_0603_1608Metric_Pad1.08x0.95mm_HandSolder, symbol Device:C_Small
- added C5, C6, C7: 1uF, Capacitor_SMD:C_0603_1608Metric_Pad1.08x0.95mm_HandSolder, symbol Device:C_Small
- added TP1, TP10, TP11, TP12, TP13, TP14, TP15, TP16, TP17, TP18, TP19, TP2, TP20, TP3, TP4, TP5, TP6, TP7, TP8, TP9: TestPoint, TestPoint:TestPoint_Pad_D2.0mm, symbol Connector:TestPoint
- A1: footprint PCM_SL_Development_Boards:raspberry_pi_pico_THT -> Module:RaspberryPi_Pico_Common_THT
- ADC1: renamed from ADC0; footprint ADC:SOP65P640X120-28N -> Package_SO:TSSOP-28_4.4x9.7mm_P0.65mm
- ADC2: renamed from ADC1; footprint ADC:SOP65P640X120-28N -> Package_SO:TSSOP-28_4.4x9.7mm_P0.65mm
- ADC3: renamed from ADC2; footprint ADC:SOP65P640X120-28N -> Package_SO:TSSOP-28_4.4x9.7mm_P0.65mm
- C10: renamed from C17; footprint Capacitor_SMD:C_1206_3216Metric_Pad1.33x1.80mm_HandSolder -> Capacitor_SMD:C_0603_1608Metric_Pad1.08x0.95mm_HandSolder
- C11: renamed from C19; footprint Capacitor_SMD:C_1206_3216Metric_Pad1.33x1.80mm_HandSolder -> Capacitor_SMD:C_0603_1608Metric_Pad1.08x0.95mm_HandSolder
- C12: renamed from C14; footprint Capacitor_SMD:C_1206_3216Metric_Pad1.33x1.80mm_HandSolder -> Capacitor_SMD:C_0603_1608Metric_Pad1.08x0.95mm_HandSolder
- C13: renamed from C18; footprint Capacitor_SMD:C_1206_3216Metric_Pad1.33x1.80mm_HandSolder -> Capacitor_SMD:C_0603_1608Metric_Pad1.08x0.95mm_HandSolder
- C3: renamed from C13; footprint Capacitor_SMD:C_1206_3216Metric_Pad1.33x1.80mm_HandSolder -> Capacitor_SMD:C_0603_1608Metric_Pad1.08x0.95mm_HandSolder
- C4: renamed from C12; footprint Capacitor_SMD:C_1206_3216Metric_Pad1.33x1.80mm_HandSolder -> Capacitor_SMD:C_0603_1608Metric_Pad1.08x0.95mm_HandSolder
- C8: renamed from C15; footprint Capacitor_SMD:C_1206_3216Metric_Pad1.33x1.80mm_HandSolder -> Capacitor_SMD:C_0603_1608Metric_Pad1.08x0.95mm_HandSolder
- C9: renamed from C16; footprint Capacitor_SMD:C_1206_3216Metric_Pad1.33x1.80mm_HandSolder -> Capacitor_SMD:C_0603_1608Metric_Pad1.08x0.95mm_HandSolder
- IC1: footprint DAC:SOP65P640X120-20N -> Package_SO:TSSOP-20_4.4x6.5mm_P0.65mm
- R1: footprint Resistor_SMD:R_1206_3216Metric_Pad1.30x1.75mm_HandSolder -> Resistor_SMD:R_0603_1608Metric_Pad0.98x0.95mm_HandSolder
- R2: renamed from R8; footprint Resistor_SMD:R_1206_3216Metric_Pad1.30x1.75mm_HandSolder -> Resistor_SMD:R_0603_1608Metric_Pad0.98x0.95mm_HandSolder
- R3: renamed from R10; footprint Resistor_SMD:R_1206_3216Metric_Pad1.30x1.75mm_HandSolder -> Resistor_SMD:R_0603_1608Metric_Pad0.98x0.95mm_HandSolder
- R4: renamed from R9; footprint Resistor_SMD:R_1206_3216Metric_Pad1.30x1.75mm_HandSolder -> Resistor_SMD:R_0603_1608Metric_Pad0.98x0.95mm_HandSolder
- renumbered J2 to J1
Connections:
- net +12V: now also TP1.1
- net +3V3: now also TP2.1
- net +5V: now also C1.1, C2.2
- net ADC0_CS: now also TP20.1
- net ADC0_DRDY: now also TP19.1
- net ADC_NTC: now also TP15.1
- net ADIM_0: now also TP9.1
- net ADIM_1: now also TP10.1
- net ADIM_2: now also TP11.1
- net ADIM_3: now also TP12.1
- net ADIM_4: now also TP13.1
- net ADIM_5: now also TP14.1
- net GND: now also C1.2, C2.1, C5.1, C6.1, C7.1
- net PWM_0: now also TP3.1
- net PWM_1: now also TP4.1
- net PWM_2: now also TP5.1
- net PWM_3: now also TP6.1
- net PWM_4: now also TP7.1
- net PWM_5: now also TP8.1
- net SPI0_MISO: now also TP18.1
- net SPI0_MOSI: now also TP17.1
- net SPI0_SCL: now also TP16.1
- net at ADC3.9 (VREFOUT): now also C6.2
- net at ADC2.9 (VREFOUT): now also C7.2
- net at ADC1.9 (VREFOUT): now also C5.2
Other:
- added sheet Micro_SD (Micro_SD.kicad_sch)
- added sheet Power_supply (Power_supply.kicad_sch)
- note removed: "tu tez capy"
- moved on the sheet: ADC1, ADC2, ADC3, C10, C11, C12, C13, C3, C4, C8, C9, IC1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

Commit message: wip
Parts:
- added H1, H2, H3, H4: MountingHole, MountingHole:MountingHole_3.2mm_M3, symbol Mechanical:MountingHole
- J1: footprint Connector_Samtec_HPM_THT:Samtec_HPM-02-01-x-S_Straight_1x02_Pitch5.08mm -> TerminalBlock:TerminalBlock_bornier-2_P5.08mm
- renumbered TP9 to TP10, TP10 to TP11, TP11 to TP12, TP12 to TP13, TP13 to TP14, TP14 to TP15, TP15 to TP3, TP3 to TP4, TP4 to TP5, TP5 to TP6, TP6 to TP7, TP7 to TP8, TP8 to TP9
Connections:
- net ADC2_CS: now also A1.12 (GP9); no longer A1.22 (GP17)
- net DAC_CS: now also A1.17 (GP13); no longer A1.12 (GP9)
- net I_LED_0: now also ADC1.17 (AIN2/IEXC/GPIO2); no longer ADC1.12 (AIN1/IEXC)
- net I_LED_1: now also ADC1.12 (AIN1/IEXC); no longer ADC1.18 (AIN3/IEXC/GPIO3)
- net I_LED_11: now also ADC3.15 (AIN6/IEXC/GPIO6); no longer ADC3.16 (AIN7/IEXC/GPIO7)
- net I_LED_3: now also ADC1.15 (AIN6/IEXC/GPIO6); no longer ADC1.16 (AIN7/IEXC/GPIO7)
- net I_LED_4: now also ADC2.17 (AIN2/IEXC/GPIO2); no longer ADC2.12 (AIN1/IEXC)
- net I_LED_5: now also ADC2.12 (AIN1/IEXC); no longer ADC2.18 (AIN3/IEXC/GPIO3)
- net I_LED_7: now also ADC2.15 (AIN6/IEXC/GPIO6); no longer ADC2.16 (AIN7/IEXC/GPIO7)
- net I_LED_8: now also ADC3.17 (AIN2/IEXC/GPIO2); no longer ADC3.12 (AIN1/IEXC)
- net I_LED_9: now also ADC3.12 (AIN1/IEXC); no longer ADC3.18 (AIN3/IEXC/GPIO3)
- net LED_0: now also ADC1.18 (AIN3/IEXC/GPIO3); no longer ADC1.11 (AIN0/IEXC)
- net LED_1: now also ADC1.11 (AIN0/IEXC); no longer ADC1.17 (AIN2/IEXC/GPIO2)
- net LED_11: now also ADC3.16 (AIN7/IEXC/GPIO7); no longer ADC3.15 (AIN6/IEXC/GPIO6)
- net LED_3: now also ADC1.16 (AIN7/IEXC/GPIO7); no longer ADC1.15 (AIN6/IEXC/GPIO6)
- net LED_4: now also ADC2.18 (AIN3/IEXC/GPIO3); no longer ADC2.11 (AIN0/IEXC)
- net LED_5: now also ADC2.11 (AIN0/IEXC); no longer ADC2.17 (AIN2/IEXC/GPIO2)
- net LED_7: now also ADC2.16 (AIN7/IEXC/GPIO7); no longer ADC2.15 (AIN6/IEXC/GPIO6)
- net LED_8: now also ADC3.18 (AIN3/IEXC/GPIO3); no longer ADC3.11 (AIN0/IEXC)
- net LED_9: now also ADC3.11 (AIN0/IEXC); no longer ADC3.17 (AIN2/IEXC/GPIO2)
- net SD_CS: now also A1.22 (GP17); no longer A1.17 (GP13)
