File: Power_supply.kicad_sch (KiCad schematic)
At the start: 16 parts, among them J2 DC_DC_Buck_converter_module, U1 TPS562201DDCR

Commit message: changing footprint for buck converter coil
Parts:
- L13: footprint footprint_lib:HPIO530-4R7 -> Inductor_SMD:L_1008_2520Metric_Pad1.43x2.20mm_HandSolder
Changed lines of the file:
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@@
 			)
 		)
-		(property "Footprint" "footprint_lib:HPIO530-4R7"
+		(property "Footprint" "Inductor_SMD:L_1008_2520Metric_Pad1.43x2.20mm_HandSolder"
 			(at 139.7 85.09 0)
 			(effects
