File: Power_supply.kicad_sch (KiCad schematic)
At the start: 16 parts, among them U1 TPS562201DDCR, U2 LM2596 BUCK MODULE

Commit message: eloleo
Parts:
- L1: footprint Inductor_SMD:L_1008_2520Metric_Pad1.43x2.20mm_HandSolder -> footprint_lib:HPIO530-4R7
Changed lines of the file:
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@@
 			)
 		)
-		(property "Footprint" "Inductor_SMD:L_1008_2520Metric_Pad1.43x2.20mm_HandSolder"
+		(property "Footprint" "footprint_lib:HPIO530-4R7"
 			(at 139.7 85.09 0)
 			(effects
