File: mgr_board.kicad_pcb (KiCad board)
At the start: 2 copper layers, 150 x 150 mm, 224 parts, among them IC1 MCP48CVB08-20E_ST, IC10 A6214KLKTR-T, IC11 A6214KLKTR-T, IC12 A6214KLKTR-T, IC13 A6214KLKTR-T, IC2 A6214KLKTR-T, IC3 A6214KLKTR-T, IC4 A6214KLKTR-T, IC5 A6214KLKTR-T, IC6 A6214KLKTR-T, IC7 A6214KLKTR-T, IC8 A6214KLKTR-T, IC9 A6214KLKTR-T, J1 Screw_Terminal_2_P5.00mm, J2 DC_DC_Buck_converter_module, J3 SD Card SPI Module, J4 Micro_SD_Card, U1 TPS562201DDCR

Commit message: wip
Parts:
- added R49: NMT, Resistor_SMD:R_0402_1005Metric, F.Cu at (55.2, 56.6)
- added R50: NMT, Resistor_SMD:R_0402_1005Metric, F.Cu at (52.7, 56.6)
- added R51: NMT, Resistor_SMD:R_0402_1005Metric, F.Cu at (60.3, 56.6)
- added R52: NMT, Resistor_SMD:R_0402_1005Metric, F.Cu at (29.8, 56.6)
- added R53: NMT, Resistor_SMD:R_0402_1005Metric, F.Cu at (27.3, 56.6)
- added R54: NMT, Resistor_SMD:R_0402_1005Metric, F.Cu at (34.9, 56.6)
- added R55: NMT, Resistor_SMD:R_0402_1005Metric, F.Cu at (22.2, 56.6)
- added R56: NMT, Resistor_SMD:R_0402_1005Metric, F.Cu at (65.4, 31.2)
- added R57: NMT, Resistor_SMD:R_0402_1005Metric, F.Cu at (47.6, 56.6)
- added R58: NMT, Resistor_SMD:R_0402_1005Metric, F.Cu at (136.7, 62.5)
- added R59: NMT, Resistor_SMD:R_0402_1005Metric, F.Cu at (87.1, 63.0)
- added R60: NMT, Resistor_SMD:R_0402_1005Metric, F.Cu at (37.3, 62.5)
- added R61: NMT, Resistor_SMD:R_0402_1005Metric, F.Cu at (110.2, 74.9)
- added R62: NMT, Resistor_SMD:R_0402_1005Metric, F.Cu at (90.3, 41.6)
- moved C77 202.6 mm to (160.8, 136.6), turned to -90 degrees
- moved C82 196.1 mm to (160.8, 158.4), turned to -90 degrees
- moved C72 189.1 mm to (134.6, 158.4), turned to -90 degrees
- moved LED8 188.6 mm to (130.0, 159.2), turned to -90 degrees
- moved C67 158.4 mm to (134.6, 136.6), turned to -90 degrees
- moved C57 151.8 mm to (110.2, 136.6), turned to -90 degrees
- moved C62 140.2 mm to (110.2, 158.4), turned to -90 degrees
- moved TH1 128.8 mm to (93.5, 148.6)
- moved C37 123.3 mm to (82.4, 136.6), turned to -90 degrees
- moved C52 103.8 mm to (82.4, 158.4), turned to -90 degrees
- moved LED13 89.6 mm to (53.1, 137.5), turned to -90 degrees
- moved C47 89.5 mm to (57.8, 158.4), turned to -90 degrees
- moved LED5 86.6 mm to (29.7, 137.5), turned to -90 degrees
- moved C42 75.5 mm to (34.3, 158.4), turned to -90 degrees
- moved C32 66.5 mm to (57.8, 136.6), turned to -90 degrees
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Connections:
- A1 pad 12: /ADC2_CS -> Net-(A1-GP9)
- A1 pad 14: /SPI1_SCL -> Net-(A1-GP10)
- A1 pad 15: /SPI1_MOSI -> Net-(A1-GP11)
- A1 pad 17: /DAC_CS -> Net-(A1-GP13)
- A1 pad 2: /ADC0_CS -> Net-(A1-GP1)
- A1 pad 22: /SD_CS -> Net-(A1-GP17)
- A1 pad 4: /SPI0_SCL -> Net-(A1-GP2)
- A1 pad 5: /SPI0_MOSI -> Net-(A1-GP3)
- A1 pad 7: /ADC1_CS -> Net-(A1-GP5)
- ADC1 pad 26: /SPI0_MISO -> Net-(ADC1-DOUT/~{DRDY})
- ADC2 pad 26: /SPI0_MISO -> Net-(ADC2-DOUT/~{DRDY})
- ADC3 pad 26: /SPI0_MISO -> Net-(ADC3-DOUT/~{DRDY})
- IC1 pad 13: /ADIM_3 -> /ADIM_2
- IC1 pad 14: /ADIM_5 -> /ADIM_4
- IC1 pad 17: /SPI1_MISO -> Net-(IC1-SDO)
- IC1 pad 6: /ADIM_4 -> /ADIM_5
- IC1 pad 7: /ADIM_2 -> /ADIM_3
- J3 pad 3: /SPI1_MISO -> /Micro_SD/SPI1_MISO
- J4 pad 7: /SPI1_MISO -> /Micro_SD/SPI1_MISO
- R1 pad 1: GND -> /ADC_NTC
- R1 pad 2: /ADC_NTC -> +3V3
- R12 pad 1: /SPI1_MISO -> /Micro_SD/SPI1_MISO
- TH1 pad 1: +3V3 -> /ADC_NTC
- TH1 pad 2: /ADC_NTC -> GND
- TP23 pad 1: /SPI1_MISO -> /Micro_SD/SPI1_MISO
Routing:
- net /ADC_NTC: track 0.00 -> 159.6 mm, vias 0 -> 6
- net /LED_11: track 39.5 -> 151.7 mm, vias 2 -> 9
- net /LED_7: track 40.3 -> 138.7 mm
- net /LED_9: track 54.8 -> 151.7 mm
- net /ADIM_4: track 0.00 -> 92.5 mm, vias 0 -> 6
- net /LED_5: track 54.4 -> 144.1 mm
- net /LED_1: track 51.8 -> 139.6 mm
- net /LED_3: track 39.5 -> 127.0 mm
- net /SPI1_MOSI: track 59.1 -> 141.1 mm, vias 4 -> 6
- net /SPI1_SCL: track 65.3 -> 147.2 mm, vias 1 -> 3
- net /SPI1_MISO: track 56.5 -> 121.6 mm, vias 1 -> 2
- net /ADIM_5: track 0.00 -> 64.3 mm, vias 0 -> 4
- net /ADIM_0: track 0.00 -> 60.8 mm, vias 0 -> 4
- net /LED_6: track 58.4 -> 104.7 mm, vias 2 -> 4
- net /ADIM_2: track 0.00 -> 45.3 mm, vias 0 -> 2
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
Commit message: wip
Parts:
- removed J2: DC_DC_Buck_converter_module, Connector_PinHeader_2.54mm:PinHeader_1x03_P2.54mm_Vertical
- removed TP1, TP10, TP11, TP12, TP13, TP14, TP15, TP16, TP17, TP18, TP19, TP2, TP20, TP21, TP22, TP3, TP4, TP5, TP6, TP7, TP8, TP9: TestPoint, TestPoint:TestPoint_Pad_D2.0mm
- added U2: LM2596 BUCK MODULE, footprint_lib:LM2596 DC-DC module, F.Cu at (146.8, 43.5)
- moved J1 21.4 mm to (164.1, 60.3)
- moved C1 15.8 mm to (23.1, 29.8)
- moved C2 15.7 mm to (23.1, 31.5)
- moved R5 10.7 mm to (162.6, 36.4)
- moved C14 10.7 mm to (160.3, 43.4)
- moved C16 10.7 mm to (160.5, 40.0)
- moved C17 10.7 mm to (157.2, 34.8)
- moved C18 10.7 mm to (153.4, 43.1)
- moved C19 10.7 mm to (153.2, 41.1)
- moved C20 10.7 mm to (153.2, 39.4)
- moved R6 10.7 mm to (164.2, 36.4)
- moved R7 10.7 mm to (158.2, 30.6)
- moved R8 10.7 mm to (158.2, 32.1)
- moved U1 10.7 mm to (159.8, 35.5)
- moved C15 10.7 mm to (160.5, 41.5)
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Connections:
- J1 pad 1: GND -> +12V
- J1 pad 2: +12V -> GND
Routing:
- net +12V: track 88.5 -> 529.3 mm, vias 0 -> 74
- net +5V: track 49.7 -> 330.8 mm, vias 0 -> 4
- net +3V3: track 40.2 -> 271.0 mm, vias 0 -> 2
- net GND: track 144.5 -> 56.3 mm, vias 168 -> 1071
- net /DAC_CS: track 0.00 -> 68.4 mm, vias 0 -> 4
- net /LED_5: track 144.1 -> 158.9 mm
- net /LED_2: track 83.7 -> 96.2 mm
- net /LED_3: track 127.0 -> 139.3 mm
- net /LED_4: track 108.7 -> 120.0 mm
- net /LED_1: track 139.6 -> 148.9 mm
- net Net-(ADC1-~{RESET}): track 2.04 -> 5.14 mm
- net Net-(ADC3-~{RESET}): track 2.04 -> 4.78 mm
- net Net-(ADC2-~{RESET}): track 2.08 -> 4.53 mm
- net /LED_9: track 151.7 -> 149.7 mm
- net /PWM_4: track 82.9 -> 84.9 mm, vias 0 -> 4
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- added copper zone on B.Cu, net +12V
- added copper zone on F.Cu, net +12V
- added copper zone on F.Cu, net +5V
- added copper zone on B.Cu, net GND
- added copper zone on F.Cu, net GND
Other:
- outline, holes or cut-outs redrawn

Commit message: Commit after kicad fuckup project
Parts:
- moved C40 0.20 mm to (19.8, 82.1)
Routing:
- net +3V3: track 271.0 -> 287.0 mm, vias 2 -> 4
- net GND: track 56.3 -> 49.9 mm, vias 1071 -> 1088
- net /PWM_4: track 84.9 -> 89.8 mm
- net /SPI0_MISO: track 125.8 -> 128.4 mm
- net /PWM_5: track 60.7 -> 63.0 mm
- net /SPI0_MOSI: track 122.5 -> 124.6 mm
- net Net-(IC5-TON): track 0.00 -> 1.99 mm
- net +12V: track 529.3 -> 527.3 mm
- net Net-(IC13-VCC): track 0.00 -> 1.60 mm
- net /SPI1_MOSI: track 141.8 -> 142.8 mm
- net /SPI0_SCL: track 123.7 -> 124.7 mm
- net /SPI1_MISO: track 121.6 -> 122.4 mm
- net /ADC1_CS: track 60.2 -> 61.0 mm
- net /ADC2_DRDY: track 102.8 -> 103.5 mm
- net /ADIM_5: track 64.3 -> 63.6 mm
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- added copper zone on B.Cu, net +3V3
- added copper zone on F.Cu, net +3V3

Commit message: wip
Routing:
- net /LED_9: track 149.7 -> 148.8 mm
- net /PWM_0: track 84.6 -> 85.4 mm
- net /PWM_1: track 58.7 -> 59.5 mm
- net /I_LED_5: track 59.8 -> 60.4 mm
- net GND: vias 1088 -> 1091
Other:
- board text added: "12V"
- board text added: "GND"
