File: mgr_board.kicad_pcb (KiCad board)
At the start: 2 copper layers, 150 x 150 mm, 216 parts, among them IC1 MCP48CVB08-20E_ST, IC10 A6214KLKTR-T, IC11 A6214KLKTR-T, IC12 A6214KLKTR-T, IC13 A6214KLKTR-T, IC2 A6214KLKTR-T, IC3 A6214KLKTR-T, IC4 A6214KLKTR-T, IC5 A6214KLKTR-T, IC6 A6214KLKTR-T, IC7 A6214KLKTR-T, IC8 A6214KLKTR-T, IC9 A6214KLKTR-T, J1 Screw_Terminal_2_P5.00mm, J3 SD Card SPI Module, J4 Micro_SD_Card, U1 TPS562201DDCR, U2 LM2596 BUCK MODULE

Commit message: finished boarD
Parts:
- added C83: 100uF, Capacitor_SMD:CP_Elec_6.3x7.7, F.Cu at (91.0, 102.0)
- added C84: 100uF, Capacitor_SMD:CP_Elec_6.3x7.7, F.Cu at (80.2, 75.5)
- added TP1: TestPoint, TestPoint:TestPoint_Pad_D2.0mm, F.Cu at (160.7, 66.2)
- added TP10: TestPoint, TestPoint:TestPoint_Pad_D2.0mm, F.Cu at (98.7, 73.5)
- added TP11: TestPoint, TestPoint:TestPoint_Pad_D2.0mm, F.Cu at (102.0, 73.5)
- added TP12: TestPoint, TestPoint:TestPoint_Pad_D2.0mm, F.Cu at (108.7, 79.9)
- added TP13: TestPoint, TestPoint:TestPoint_Pad_D2.0mm, F.Cu at (114.5, 79.9)
- added TP14: TestPoint, TestPoint:TestPoint_Pad_D2.0mm, F.Cu at (116.8, 65.8)
- added TP15: TestPoint, TestPoint:TestPoint_Pad_D2.0mm, F.Cu at (116.8, 61.5)
- added TP16: TestPoint, TestPoint:TestPoint_Pad_D2.0mm, F.Cu at (132.5, 61.5)
- added TP17: TestPoint, TestPoint:TestPoint_Pad_D2.0mm, F.Cu at (135.0, 58.5)
- added TP18: TestPoint, TestPoint:TestPoint_Pad_D2.0mm, F.Cu at (138.4, 60.5)
- added TP19: TestPoint, TestPoint:TestPoint_Pad_D2.0mm, F.Cu at (36.6, 59.5)
- added TP2: TestPoint, TestPoint:TestPoint_Pad_D2.0mm, F.Cu at (29.7, 30.2)
- added TP20: TestPoint, TestPoint:TestPoint_Pad_D2.0mm, F.Cu at (22.2, 60.1)
- added TP22: TestPoint, TestPoint:TestPoint_Pad_D2.0mm, F.Cu at (104.8, 46.8)
- added TP3: TestPoint, TestPoint:TestPoint_Pad_D2.0mm, F.Cu at (42.5, 28.9)
- added TP4: TestPoint, TestPoint:TestPoint_Pad_D2.0mm, F.Cu at (25.1, 65.7)
- added TP5: TestPoint, TestPoint:TestPoint_Pad_D2.0mm, F.Cu at (29.3, 65.7)
- added TP6: TestPoint, TestPoint:TestPoint_Pad_D2.0mm, F.Cu at (47.7, 30.5)
- added TP7: TestPoint, TestPoint:TestPoint_Pad_D2.0mm, F.Cu at (52.2, 30.5)
- added TP8: TestPoint, TestPoint:TestPoint_Pad_D2.0mm, F.Cu at (55.2, 30.5)
- added TP9: TestPoint, TestPoint:TestPoint_Pad_D2.0mm, F.Cu at (58.3, 30.5)
- R7: value 54,9k -> 56k
Routing:
- net +5V: track 331.2 -> 336.6 mm
- net +3V3: track 287.0 -> 291.9 mm
- net /PWM_5: track 63.0 -> 67.9 mm
- net /PWM_3: track 55.8 -> 60.6 mm
- net /PWM_2: track 82.3 -> 86.9 mm
- net /PWM_4: track 89.8 -> 94.4 mm
- net +12V: track 527.3 -> 530.7 mm
- net /SPI0_MISO: track 128.4 -> 131.4 mm
- net /ADIM_0: track 61.1 -> 63.9 mm
- net /ADC_NTC: track 159.7 -> 162.3 mm
- net /ADIM_3: track 25.7 -> 27.9 mm, vias 2 -> 3
- net /ADC0_CS: track 22.5 -> 24.7 mm
- net /ADIM_1: track 26.1 -> 28.2 mm, vias 2 -> 3
- net /ADIM_2: track 45.7 -> 47.7 mm, vias 2 -> 3
- net /SPI0_SCL: track 124.7 -> 126.6 mm
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