File: LED_Section.kicad_sch (KiCad schematic)
At the start: 16 parts

Commit message: Changed footprints of passive elements, reviewed
Parts:
- LED1: renamed from LED12; footprint CREE_RGB_LED:XPLDCL0000000000HC6AAAE7 -> footprint_lib:XPLDCL
- LED10: renamed from LED4; footprint JR5050CWTEB50EB0000N0000001 -> footprint_lib:JR5050CWT
- LED11: renamed from LED7; footprint JR5050CWTEB50EB0000N0000001 -> footprint_lib:JR5050CWT
- LED12: renamed from LED10; footprint JR5050CWTEB50EB0000N0000001 -> footprint_lib:JR5050CWT
- LED13: renamed from LED2; footprint JR5050CWTEB50EB0000N0000001 -> footprint_lib:JR5050CWT
- LED14: renamed from LED5; footprint JR5050CWTEB50EB0000N0000001 -> footprint_lib:JR5050CWT
- LED15: renamed from LED8; footprint JR5050CWTEB50EB0000N0000001 -> footprint_lib:JR5050CWT
- LED16: renamed from LED11; footprint JR5050CWTEB50EB0000N0000001 -> footprint_lib:JR5050CWT
- LED2: renamed from LED13; footprint CREE_RGB_LED:XPLDCL0000000000HC6AAAE7 -> footprint_lib:XPLDCL
- LED3: renamed from LED14; footprint XPLDCL0000000000HC6AAAE7 -> footprint_lib:XPLDCL
- LED4: renamed from LED15; footprint XPLDCL0000000000HC6AAAE7 -> footprint_lib:XPLDCL
- LED5: renamed from LED0; footprint Cree_White_LED:JR5050CWTEB50EB0000N0000001 -> footprint_lib:JR5050CWT
- LED6: renamed from LED3; footprint JR5050CWTEB50EB0000N0000001 -> footprint_lib:JR5050CWT
- LED7: renamed from LED6; footprint JR5050CWTEB50EB0000N0000001 -> footprint_lib:JR5050CWT
- LED8: renamed from LED9; footprint JR5050CWTEB50EB0000N0000001 -> footprint_lib:JR5050CWT
- LED9: renamed from LED1; footprint Cree_White_LED:JR5050CWTEB50EB0000N0000001 -> footprint_lib:JR5050CWT
Connections:
- net LED_2: now also LED13.2 (A)
