File: hw/mgr_board.kicad_pcb (KiCad board)
At the start: 2 copper layers, 150 x 150 mm, 239 parts, among them IC1 MCP48CVB08-20E_ST, IC10 A6214KLKTR-T, IC11 A6214KLKTR-T, IC12 A6214KLKTR-T, IC13 A6214KLKTR-T, IC2 A6214KLKTR-T, IC3 A6214KLKTR-T, IC4 A6214KLKTR-T, IC5 A6214KLKTR-T, IC6 A6214KLKTR-T, IC7 A6214KLKTR-T, IC8 A6214KLKTR-T, IC9 A6214KLKTR-T, J1 Screw_Terminal_2_P5.00mm, J3 SD Card SPI Module, J4 Micro_SD_Card, U1 TPS562201DDCR, U2 LM2596 BUCK MODULE

Commit message: fixing bugs
Parts:
- moved R7 1.64 mm to (159.9, 30.6)
- moved R8 1.64 mm to (159.9, 32.1)
- moved TP5 0.70 mm to (30.0, 65.7)
- moved TP4 0.30 mm to (24.8, 65.7)
Routing:
- net +12V: track 530.7 -> 555.9 mm, vias 74 -> 60
- net GND: track 48.1 -> 56.6 mm, vias 1097 -> 1261
- net /LED_6: track 104.7 -> 108.6 mm, vias 4 -> 8
- net /LED_4: track 119.7 -> 123.5 mm
- net /LED_9: track 148.8 -> 152.6 mm
- net /LED_0: track 124.3 -> 127.1 mm, vias 4 -> 8
- net /PWM_3: track 60.6 -> 58.0 mm
- net /LED_1: track 148.3 -> 150.9 mm
- net /LED_11: track 151.3 -> 148.9 mm
- net /LED_2: track 96.2 -> 98.1 mm
- net /LED_7: track 140.7 -> 142.2 mm
- net /LED_3: track 139.3 -> 140.8 mm
- net Net-(U1-VFB): track 5.08 -> 3.65 mm
- net +5V: track 336.6 -> 335.3 mm, vias 4 -> 8
- net /LED_8: track 121.7 -> 122.9 mm
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Other:
- board text added: "JLCJLCJLCJLC"
